Commit message: align rotation convention of hip and knee with Cheetah Software

File: urdf/mini_cheetah_simple_correctedInertia.urdf (robot description, URDF)
Before this commit: robot mini_cheetah, 17 links, 16 joints
Links:
- link body: mass 3.3 -> 4.0
Joints:
- joint abduct_fl_to_thigh_fl_j: origin xyz=0.0 0.062 0.00 rpy=0.0 0.0 0.0 -> xyz=0.0 0.062 0.00 rpy=0.0 0.0 3.1415
- joint abduct_fr_to_thigh_fr_j: origin xyz=0.0 -0.062 0.00 rpy=0.0 0.0 0.0 -> xyz=0.0 -0.062 0.00 rpy=0.0 0.0 3.1415
- joint abduct_hl_to_thigh_hl_j: origin xyz=0.0 0.062 0.00 rpy=0.0 0.0 0.0 -> xyz=0.0 0.062 0.00 rpy=0.0 0.0 3.1415
- joint abduct_hr_to_thigh_hr_j: origin xyz=0.0 -0.062 0.00 rpy=0.0 0.0 0.0 -> xyz=0.0 -0.062 0.00 rpy=0.0 0.0 3.1415

Commit message: revert tuned body inertia

File: urdf/mini_cheetah_simple_correctedInertia.urdf (robot description, URDF)
Before this commit: robot mini_cheetah, 17 links, 16 joints
Links:
- link body: mass 4.0 -> 3.3
